File: conf2025badge/conf2025badge/conf2025badge.kicad_sch (KiCad schematic)
At the start: 11 parts, among them SW1 SW_PUSH, SW2 RotaryEncoder_Switch, SW3 SW_PUSH, U1 xiao, U2 RKJXV122400R

Commit message: Update
Parts:
- removed D1: LED, symbol Device:LED
- removed U2: RKJXV122400R, sglib:RKJXV122400R, symbol sglib:RKJXV122400R
- added H1, H2, H3, H4: MountingHole, foostan/kbd:M2_HOLE_v2, symbol Mechanical:MountingHole
- added R2: R, Resistor_THT:R_Axial_DIN0207_L6.3mm_D2.5mm_P10.16mm_Horizontal, symbol Device:R
- added U3: fj08k-s, sglib:FJ08K-S, symbol sglib:fj08k-s
- R1: footprint (none) -> Resistor_THT:R_Axial_DIN0207_L6.3mm_D2.5mm_P10.16mm_Horizontal
- renumbered SW2 to SW5
Connections:
- net 3V3: now reaches R1.1
- net 3V3: now also LED1.1 (VDD), LED2.1 (VDD), OL1.3 (VCC), U1.12 (3V3), R2.1, U3.3 (VR1-3), U3.4 (VR2-1)
- net SDA: now reaches R1.2
- net SDA: now also OL1.1 (SDA), U1.5 (A8_SDA)
- net SCL: now reaches OL1.2 (SCL)
- net SCL: now also U1.6 (A9_SCL), R2.2
- net GND: now reaches OL1.4 (GND)
- net GND: now also BZ1.2 (-), LED1.3 (VSS), LED2.3 (VSS), SW1.2, SW3.2, SW5.C, SW5.S2, U1.13 (GND), U3.1 (VR1-1), U3.6 (VR2-3)
- net BUZZER: now reaches BZ1.1 (+)
- net BUZZER: now also U1.8 (B9_RX)
- net at LED1.2 (DOUT): now also LED2.4 (DIN)
- net SK6812MINI-E: now reaches LED1.4 (DIN)
- net SK6812MINI-E: now also U1.7 (B8_TX)
- net VR_X: now reaches U1.1 (A2)
- net VR_X: now also U3.2 (VR1-2)
- net ROT_B: now reaches U1.10 (A5_MISO)
- net ROT_B: now also SW5.B
- net ROT_A: now reaches U1.11 (A6_MOSI)
- net ROT_A: now also SW5.A
- net VR_Y: now reaches U1.2 (A4)
- net VR_Y: now also U3.5 (VR2-2)
- net SW_1: now reaches U1.3 (A10)
- net SW_1: now also SW1.1
- net SW_2: now reaches U1.4 (A11)
- net SW_2: now also SW3.1
- net ROT_BTN: now reaches U1.9 (A7_SCK)
- net ROT_BTN: now also SW5.S1
- no-connect marks 0 -> 8
Other:
- moved on the sheet: LED1, LED2, SW5
